File: dac.kicad_sch (KiCad schematic)
At the start: 19 parts, among them U401 SN74LVC1G04DBVR, U403 AD567xR

Commit message: update datasheets and footprint references
Parts:
- C302, C303, C401, C405, C406: footprint pss:C_0805_2012Metric_Pad1.18x1.45mm_HandSolder -> enclosure:C_0805_2012Metric_Pad1.18x1.45mm_HandSolder
- C407: footprint pss:C_1210_3225Metric_Pad1.33x2.70mm_HandSolder -> enclosure:C_1210_3225Metric_Pad1.33x2.70mm_HandSolder
- JP401: footprint pss:SolderJumper-3_P1.3mm_Bridged12-Soldermask-Paste_RoundedPad1.0x1.5mm -> enclosure:SolderJumper-3_P1.3mm_Bridged12-Soldermask-Paste_RoundedPad1.0x1.5mm
- R301, R302: footprint pss:R_1210_3225Metric_Pad1.30x2.65mm_HandSolder -> enclosure:R_1210_3225Metric_Pad1.30x2.65mm_HandSolder
- TP301, TP302, TP303, TP304, TP305, TP306, TP307, TP308: footprint pss:TP_0805_2012Metric -> enclosure:TP_0805_2012Metric
- U401: footprint pss:SOT-23-5_HandSoldering -> enclosure:SOT-23-5_HandSoldering
- U403: footprint pss:TSSOP-20_4.4x6.5mm_P0.65mm -> enclosure:TSSOP-20_4.4x6.5mm_P0.65mm
Changed lines of the file:
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@@
 			)
 		)
-		(property "Footprint" "pss:SOT-23-5_HandSoldering"
+		(property "Footprint" "enclosure:SOT-23-5_HandSoldering"
 			(at 67.31 83.82 0)
 			(effects
@@
 			)
 		)
-		(property "Footprint" "pss:R_1210_3225Metric_Pad1.30x2.65mm_HandSolder"
+		(property "Footprint" "enclosure:R_1210_3225Metric_Pad1.30x2.65mm_HandSolder"
 			(at 82.55 77.978 90)
 			(effects
@@
 			)
 		)
-		(property "Footprint" "pss:TP_0805_2012Metric"
+		(property "Footprint" "enclosure:TP_0805_2012Metric"
 			(at 213.36 116.84 0)
 			(effects
@@
 			)
 		)
-		(property "Footprint" "pss:C_1210_3225Metric_Pad1.33x2.70mm_HandSolder"
+		(property "Footprint" "enclosure:C_1210_3225Metric_Pad1.33x2.70mm_HandSolder"
 			(at 176.8348 64.77 0)
 			(effects
@@
 			)
 		)
-		(property "Footprint" "pss:TP_0805_2012Metric"
+		(property "Footprint" "enclosure:TP_0805_2012Metric"
 			(at 200.66 104.14 0)
 			(effects
@@
 			)
 		)
-		(property "Footprint" "pss:R_1210_3225Metric_Pad1.30x2.65mm_HandSolder"
+		(property "Footprint" "enclosure:R_1210_3225Metric_Pad1.30x2.65mm_HandSolder"
 			(at 82.55 103.378 90)
 			(effects
@@
 			)
 		)
-		(property "Footprint" "pss:TP_0805_2012Metric"
+		(property "Footprint" "enclosure:TP_0805_2012Metric"
 			(at 210.82 114.3 0)
 			(effects
@@
 			)
 		)
-		(property "Footprint" "pss:C_0805_2012Metric_Pad1.18x1.45mm_HandSolder"
+		(property "Footprint" "enclosure:C_0805_2012Metric_Pad1.18x1.45mm_HandSolder"
 			(at 172.72 93.0148 0)
 			(effects
@@
 			)
 		)
-		(property "Footprint" "pss:C_0805_2012Metric_Pad1.18x1.45mm_HandSolder"
+		(property "Footprint" "enclosure:C_0805_2012Metric_Pad1.18x1.45mm_HandSolder"
 			(at 52.3748 62.23 0)
 			(effects
@@
 			)
 		)
-		(property "Footprint" "pss:TSSOP-20_4.4x6.5mm_P0.65mm"
+		(property "Footprint" "enclosure:TSSOP-20_4.4x6.5mm_P0.65mm"
 			(at 148.59 137.16 0)
 			(effects
@@
 			)
 		)
-		(property "Footprint" "pss:TP_0805_2012Metric"
+		(property "Footprint" "enclosure:TP_0805_2012Metric"
 			(at 205.74 109.22 0)
 			(effects
@@
 			)
 		)
-		(property "Footprint" "pss:TP_0805_2012Metric"
+		(property "Footprint" "enclosure:TP_0805_2012Metric"
 			(at 208.28 111.76 0)
 			(effects
@@
 			)
 		)
-		(property "Footprint" "pss:C_0805_2012Metric_Pad1.18x1.45mm_HandSolder"
+		(property "Footprint" "enclosure:C_0805_2012Metric_Pad1.18x1.45mm_HandSolder"
 			(at 161.5948 64.77 0)
 			(effects
@@
 			)
 		)
-		(property "Footprint" "pss:TP_0805_2012Metric"
+		(property "Footprint" "enclosure:TP_0805_2012Metric"
 			(at 203.2 106.68 0)
 			(effects
@@
 			)
 		)
-		(property "Footprint" "pss:SolderJumper-3_P1.3mm_Bridged12-Soldermask-Paste_RoundedPad1.0x1.5mm"
+		(property "Footprint" "enclosure:SolderJumper-3_P1.3mm_Bridged12-Soldermask-Paste_RoundedPad1.0x1.5mm"
 			(at 114.3 111.76 0)
 			(effects
@@
 			)
 		)
-		(property "Footprint" "pss:C_0805_2012Metric_Pad1.18x1.45mm_HandSolder"
+		(property "Footprint" "enclosure:C_0805_2012Metric_Pad1.18x1.45mm_HandSolder"
 			(at 75.2348 104.14 0)
 			(effects
@@
 			)
 		)
-		(property "Footprint" "pss:C_0805_2012Metric_Pad1.18x1.45mm_HandSolder"
+		(property "Footprint" "enclosure:C_0805_2012Metric_Pad1.18x1.45mm_HandSolder"
 			(at 87.9348 78.74 0)
 			(effects
@@
 			)
 		)
-		(property "Footprint" "pss:TP_0805_2012Metric"
+		(property "Footprint" "enclosure:TP_0805_2012Metric"
 			(at 198.12 101.6 0)
 			(effects
@@
 			)
 		)
-		(property "Footprint" "pss:TP_0805_2012Metric"
+		(property "Footprint" "enclosure:TP_0805_2012Metric"
 			(at 195.58 99.06 0)
 			(effects
