File: digital-interface.kicad_sch (KiCad schematic)
At the start: 37 parts, among them U701 Si8641BD-B-IS2, U702 R05C05TE05S

Commit message: add digital-interface sub layout
Connections:
- net sdo_iso_pin: now reaches R205.2, U701.6 (A4)
- net ~{cs_pin}: now reaches R208.1, U701.14 (B1)
- net sckl_pin: now reaches R209.1, U701.13 (B2)
- net sdi_pin: now reaches R210.1, U701.12 (B3)
Other:
- moved on the sheet: R205
Changed lines of the file:
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@@
 	(wire
 		(pts
-			(xy 151.13 76.2) (xy 156.21 76.2)
+			(xy 147.32 76.2) (xy 156.21 76.2)
 		)
 		(stroke
@@
 	(wire
 		(pts
-			(xy 138.43 76.2) (xy 143.51 76.2)
+			(xy 138.43 76.2) (xy 139.7 76.2)
 		)
 		(stroke
@@
 			(width 0)
 			(type default)
+		)
+	)
+	(label "sckl_pin"
+		(at 179.07 71.12 0)
+		(fields_autoplaced yes)
+		(effects
+			(font
+				(size 1.27 1.27)
+			)
+			(justify left bottom)
+		)
+	)
+	(label "sdo_iso_pin"
+		(at 147.32 76.2 0)
+		(fields_autoplaced yes)
+		(effects
+			(font
+				(size 1.016 1.016)
+			)
+			(justify left bottom)
+		)
+	)
+	(label "~{cs_pin}"
+		(at 179.07 68.58 0)
+		(fields_autoplaced yes)
+		(effects
+			(font
+				(size 1.27 1.27)
+			)
+			(justify left bottom)
+		)
+	)
+	(label "sdi_pin"
+		(at 179.07 73.66 0)
+		(fields_autoplaced yes)
+		(effects
+			(font
+				(size 1.27 1.27)
+			)
+			(justify left bottom)
 		)
 	)
@@
 	(symbol
 		(lib_id "enclosure:R")
-		(at 147.32 76.2 90)
+		(at 143.51 76.2 90)
 		(mirror x)
 		(unit 1)
@@
 		(dnp no)
 		(property "Reference" "R205"
-			(at 147.32 81.28 90)
+			(at 143.51 81.28 90)
 			(effects
 				(font
@@
 		)
 		(property "Value" "100"
-			(at 147.32 78.74 90)
+			(at 143.51 78.74 90)
 			(effects
 				(font
@@
 		)
 		(property "Footprint" "enclosure:R_1210_3225Metric_Pad1.30x2.65mm_HandSolder"
-			(at 147.32 74.422 90)
+			(at 143.51 74.422 90)
 			(effects
 				(font
@@
 		)
 		(property "Datasheet" "./datasheet/R_SMD_Yageo.pdf"
-			(at 147.32 76.2 0)
+			(at 143.51 76.2 0)
 			(effects
 				(font
@@
 		)
 		(property "Description" "Resistor"
-			(at 147.32 76.2 0)
+			(at 143.51 76.2 0)
 			(effects
 				(font
@@
 		)
 		(property "MPN" "RC1210FR-07100RL"
-			(at 147.32 76.2 0)
+			(at 143.51 76.2 0)
 			(effects
 				(font
@@
 		)
 		(property "VPN" "603-RC1210FR-07100RL"
-			(at 147.32 76.2 0)
-			(effects
-				(font
+			(at 143.51 76.2 0)
+			(effects
+				(font
