File: power.kicad_sch (KiCad schematic)
At the start: 26 parts, among them U1001 MC7805, U1002 MC7812

Commit message: add enclosure output connectors
Parts:
- renumbered C1005 to C1001, C1001 to C1002, C1002 to C1003, C1003 to C1004, C1004 to C1005
Changed lines of the file:
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@@
 	(title_block
 		(title "Power Supply Sink")
-		(date "2025-02-20")
-		(rev "0.5.0")
+		(date "2025-02-21")
+		(rev "1.0.0")
 		(company "Open Battery Tester")
 		(comment 1 "Power")
@@
 		(on_board yes)
 		(dnp no)
-		(property "Reference" "C1005"
+		(property "Reference" "C1001"
 			(at 110.49 65.1509 0)
 			(effects
@@
 			(project "enclosure"
 				(path "/8ec0899b-9d7b-491d-933a-49b74b34a0df/f6df2627-821f-46ca-b36c-d1d3b4f0e28f"
-					(reference "C1005")
+					(reference "C1001")
 					(unit 1)
 				)
@@
 		(on_board yes)
 		(dnp no)
-		(property "Reference" "C1004"
+		(property "Reference" "C1005"
 			(at 205.74 120.6501 0)
 			(effects
@@
 			(project "enclosure"
 				(path "/8ec0899b-9d7b-491d-933a-49b74b34a0df/f6df2627-821f-46ca-b36c-d1d3b4f0e28f"
-					(reference "C1004")
+					(reference "C1005")
 					(unit 1)
 				)
@@
 		(on_board yes)
 		(dnp no)
-		(property "Reference" "C1001"
+		(property "Reference" "C1002"
 			(at 168.91 69.8501 0)
 			(effects
@@
 			(project "enclosure"
 				(path "/8ec0899b-9d7b-491d-933a-49b74b34a0df/f6df2627-821f-46ca-b36c-d1d3b4f0e28f"
-					(reference "C1001")
+					(reference "C1002")
 					(unit 1)
 				)
@@
 		(on_board yes)
 		(dnp no)
-		(property "Reference" "C1002"
+		(property "Reference" "C1003"
 			(at 168.91 120.6501 0)
 			(effects
@@
 			(project "enclosure"
 				(path "/8ec0899b-9d7b-491d-933a-49b74b34a0df/f6df2627-821f-46ca-b36c-d1d3b4f0e28f"
-					(reference "C1002")
+					(reference "C1003")
 					(unit 1)
 				)
@@
 		(on_board yes)
 		(dnp no)
-		(property "Reference" "C1003"
+		(property "Reference" "C1004"
 			(at 205.74 69.8501 0)
 			(effects
@@
 			(project "enclosure"
 				(path "/8ec0899b-9d7b-491d-933a-49b74b34a0df/f6df2627-821f-46ca-b36c-d1d3b4f0e28f"
-					(reference "C1003")
+					(reference "C1004")
 					(unit 1)
 				)

Commit message: add increased current capacity for 12V power rail
Parts:
- added Q1001: DPLS350E, pss:SOT-223-3_TabPin2, symbol pss:Q_PNP_BCE
- added R1001: 5R9, pss:R_1210_3225Metric_Pad1.30x2.65mm_HandSolder, symbol enclosure:R
- C1004, C1005: value 1u -> 10u; footprint pss:C_0603_1608Metric_Pad1.08x0.95mm_HandSolder -> pss:C_1210_3225Metric_Pad1.33x2.70mm_HandSolder; MPN C0603C105K4RACTU -> C1210C106K3RACTU; VPN 80-C0603C105K4R -> 80-C1210C106K3R
Connections:
- net +12VA: now also Q1001.2 (C)
- net +24V: now also Q1001.3 (E), R1001.1; no longer C1003.2, D1004.1 (K), U1002.1 (IN)
- new net: C1003.2, D1004.1 (K), Q1001.1 (B), R1001.2, U1002.1 (IN)
Other:
- moved on the sheet: C1003, D1004, TP1008, TP1009, U1002

Commit message: fix symbol library link
Parts:
- Q1001: symbol pss:Q_PNP_BCE -> enclosure:Q_PNP_BCE
Changed lines of the file:
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@@
 		(title "Power Supply Sink")
 		(date "2025-02-21")
-		(rev "1.1.0")
+		(rev "1.1.1")
 		(company "Open Battery Tester")
 		(comment 1 "Power")
@@
 	)
 	(symbol
-		(lib_id "pss:Q_PNP_BCE")
+		(lib_id "enclosure:Q_PNP_BCE")
 		(at 172.72 116.84 270)
 		(mirror x)

Commit message: update datasheets and footprint references
Parts:
- C1001: footprint Capacitor_SMD:CP_Elec_10x10 -> enclosure:CP_Elec_10x10
- C1002, C1003: footprint pss:C_0603_1608Metric_Pad1.08x0.95mm_HandSolder -> enclosure:C_0603_1608Metric_Pad1.08x0.95mm_HandSolder
- C1004, C1005: footprint pss:C_1210_3225Metric_Pad1.33x2.70mm_HandSolder -> enclosure:C_1210_3225Metric_Pad1.33x2.70mm_HandSolder
- D1001: footprint pss:D_SOD-323_HandSoldering -> enclosure:D_SOD-323_HandSoldering
- D1002, D1003, D1004: footprint pss:D_SOD-123 -> enclosure:D_SOD-123
- F1002: footprint pss:FuseHolder_Blade_ATO_Littelfuse_FLR_178.6165 -> enclosure:FuseHolder_Blade_ATO_Littelfuse_FLR_178.6165
- JP1001, JP1002, JP1003, JP1004: footprint pss:SolderJumper-2_P1.3mm_Open_RoundedPad1.0x1.5mm -> enclosure:SolderJumper-2_P1.3mm_Open_RoundedPad1.0x1.5mm
- Q1001: footprint pss:SOT-223-3_TabPin2 -> enclosure:SOT-223-3_TabPin2
- R1001: footprint pss:R_1210_3225Metric_Pad1.30x2.65mm_HandSolder -> enclosure:R_1210_3225Metric_Pad1.30x2.65mm_HandSolder
- TP1001, TP1002, TP1003, TP1004, TP1005, TP1006, TP1007, TP1008, TP1009: footprint pss:TP_0805_2012Metric -> enclosure:TP_0805_2012Metric
- U1001, U1002: footprint pss:TO-252-2 -> enclosure:TO-252-2
Changed lines of the file:
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@@
 			)
 		)
-		(property "Footprint" "pss:SolderJumper-2_P1.3mm_Open_RoundedPad1.0x1.5mm"
+		(property "Footprint" "enclosure:SolderJumper-2_P1.3mm_Open_RoundedPad1.0x1.5mm"
 			(at 63.5 152.4 0)
 			(effects
@@
 			)
 		)
-		(property "Footprint" "pss:TO-252-2"
+		(property "Footprint" "enclosure:TO-252-2"
 			(at 191.135 143.51 0)
 			(effects
@@
 			)
 		)
-		(property "Footprint" "Capacitor_SMD:CP_Elec_10x10"
+		(property "Footprint" "enclosure:CP_Elec_10x10"
 			(at 113.3348 71.12 0)
 			(effects
@@
 			)
 		)
-		(property "Footprint" "pss:D_SOD-123"
+		(property "Footprint" "enclosure:D_SOD-123"
 			(at 190.5 127 0)
 			(effects
@@
 			)
 		)
-		(property "Footprint" "pss:TP_0805_2012Metric"
+		(property "Footprint" "enclosure:TP_0805_2012Metric"
 			(at 119.38 59.69 0)
 			(effects
@@
 			)
 		)
-		(property "Footprint" "pss:TP_0805_2012Metric"
+		(property "Footprint" "enclosure:TP_0805_2012Metric"
 			(at 228.6 113.03 0)
 			(effects
@@
 			)
 		)
-		(property "Footprint" "pss:C_0603_1608Metric_Pad1.08x0.95mm_HandSolder"
+		(property "Footprint" "enclosure:C_0603_1608Metric_Pad1.08x0.95mm_HandSolder"
 			(at 171.7548 64.77 0)
 			(effects
@@
 			)
 		)
-		(property "Footprint" "pss:D_SOD-323_HandSoldering"
+		(property "Footprint" "enclosure:D_SOD-323_HandSoldering"
 			(at 66.04 67.31 0)
 			(effects
@@
 			)
 		)
-		(property "Footprint" "pss:TP_0805_2012Metric"
+		(property "Footprint" "enclosure:TP_0805_2012Metric"
 			(at 71.12 60.96 0)
 			(effects
@@
 			)
 		)
-		(property "Footprint" "pss:D_SOD-123"
+		(property "Footprint" "enclosure:D_SOD-123"
 			(at 190.5 50.8 0)
 			(effects
@@
 			)
 		)
-		(property "Footprint" "pss:C_0603_1608Metric_Pad1.08x0.95mm_HandSolder"
+		(property "Footprint" "enclosure:C_0603_1608Metric_Pad1.08x0.95mm_HandSolder"
 			(at 171.7548 140.97 0)
 			(effects
@@
 			)
 		)
-		(property "Footprint" "pss:TP_0805_2012Metric"
+		(property "Footprint" "enclosure:TP_0805_2012Metric"
 			(at 81.28 127 0)
 			(effects
@@
 			)
 		)
-		(property "Footprint" "pss:TP_0805_2012Metric"
+		(property "Footprint" "enclosure:TP_0805_2012Metric"
 			(at 60.96 73.66 0)
 			(effects
@@
 			)
 		)
-		(property "Footprint" "pss:SolderJumper-2_P1.3mm_Open_RoundedPad1.0x1.5mm"
+		(property "Footprint" "enclosure:SolderJumper-2_P1.3mm_Open_RoundedPad1.0x1.5mm"
 			(at 63.5 127 0)
 			(effects
@@
 			)
 		)
-		(property "Footprint" "pss:R_1210_3225Metric_Pad1.30x2.65mm_HandSolder"
+		(property "Footprint" "enclosure:R_1210_3225Metric_Pad1.30x2.65mm_HandSolder"
 			(at 158.75 128.778 90)
 			(effects
@@
 			)
 		)
-		(property "Footprint" "pss:TO-252-2"
+		(property "Footprint" "enclosure:TO-252-2"
 			(at 191.135 67.31 0)
 			(effects
@@
 			)
 		)
-		(property "Footprint" "pss:FuseHolder_Blade_ATO_Littelfuse_FLR_178.6165"
+		(property "Footprint" "enclosure:FuseHolder_Blade_ATO_Littelfuse_FLR_178.6165"
 			(at 91.44 59.182 90)
 			(effects
@@
 			)
 		)
-		(property "Footprint" "pss:D_SOD-123"
+		(property "Footprint" "enclosure:D_SOD-123"
 			(at 127 67.31 0)
 			(effects
@@
 			)
 		)
-		(property "Footprint" "pss:SolderJumper-2_P1.3mm_Open_RoundedPad1.0x1.5mm"
+		(property "Footprint" "enclosure:SolderJumper-2_P1.3mm_Open_RoundedPad1.0x1.5mm"
 			(at 63.5 165.1 0)
 			(effects
@@
 			)
 		)
-		(property "Footprint" "pss:TP_0805_2012Metric"
+		(property "Footprint" "enclosure:TP_0805_2012Metric"
 			(at 81.28 165.1 0)
 			(effects
@@
 			)
 		)
-		(property "Footprint" "pss:TP_0805_2012Metric"
+		(property "Footprint" "enclosure:TP_0805_2012Metric"
 			(at 81.28 152.4 0)
 			(effects
@@
 			)
 		)
-		(property "Footprint" "pss:TP_0805_2012Metric"
+		(property "Footprint" "enclosure:TP_0805_2012Metric"
 			(at 228.6 62.23 0)
 			(effects
@@
 			)
 		)
-		(property "Footprint" "pss:SOT-223-3_TabPin2"
+		(property "Footprint" "enclosure:SOT-223-3_TabPin2"
 			(at 175.26 111.76 0)
 			(effects
@@
 			)
 		)
-		(property "Footprint" "pss:SolderJumper-2_P1.3mm_Open_RoundedPad1.0x1.5mm"
+		(property "Footprint" "enclosure:SolderJumper-2_P1.3mm_Open_RoundedPad1.0x1.5mm"
 			(at 63.5 139.7 0)
 			(effects
@@
 			)
 		)
-		(property "Footprint" "pss:C_1210_3225Metric_Pad1.33x2.70mm_HandSolder"
+		(property "Footprint" "enclosure:C_1210_3225Metric_Pad1.33x2.70mm_HandSolder"
 			(at 208.5848 140.97 0)
 			(effects
@@
 			)
 		)
-		(property "Footprint" "pss:TP_0805_2012Metric"
+		(property "Footprint" "enclosure:TP_0805_2012Metric"
 			(at 81.28 139.7 0)
 			(effects
@@
 			)
 		)
-		(property "Footprint" "pss:C_1210_3225Metric_Pad1.33x2.70mm_HandSolder"
+		(property "Footprint" "enclosure:C_1210_3225Metric_Pad1.33x2.70mm_HandSolder"
 			(at 208.5848 64.77 0)
 			(effects

Commit message: fix netnaming collsion
Connections:
- net +24V: no longer D1001.2 (A2), F1001.1, F1002.2, TP1001.1
- new net IN: D1001.2 (A2), F1001.1, F1002.2, TP1001.1
Changed lines of the file:
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@@
 		)
 	)
-	(hierarchical_label "+24V"
+	(hierarchical_label "IN"
 		(shape input)
 		(at 53.34 60.96 180)

Commit message: add dac sub-layout
Parts:
- removed TP1003, TP1004, TP1005, TP1006: ~, enclosure:TP_0805_2012Metric, symbol enclosure:TestPoint

Commit message: fix wrong fuse in bom
Parts:
- F1001: MPN 0287030.PXCN -> 0287010.PXCN; VPN 576-0287030.PXCN -> 576-0287010.PXCN
Changed lines of the file:
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@@
 			)
 		)
-		(property "MPN" "0287030.PXCN"
+		(property "MPN" "0287010.PXCN"
 			(at 91.44 60.96 0)
 			(effects
@@
 			)
 		)
-		(property "VPN" "576-0287030.PXCN"
+		(property "VPN" "576-0287010.PXCN"
 			(at 91.44 60.96 0)
 			(effects
